Commit message: Añadi funciones para el lidar

File: src/mtrb_description/urdf/mtrb.urdf.xacro (robot description, xacro)
@@ -9,5 +9,5 @@
   <xacro:arg name="lidar_y"     default="0.0"/>
   <xacro:arg name="lidar_z"     default="0.1"/>
-  <xacro:arg name="lidar_yaw"   default="0.0"/>
+  <xacro:arg name="lidar_yaw"   default="${pi}"/>  <!-- sllidar_ros2: C1 triangle to the front -->
   <xacro:include filename="$(find mtrb_description)/urdf/sensors/lidar.urdf.xacro"/>
   <xacro:unless value="$(arg lidar_only)">

File: src/mtrb_description/urdf/sensors/lidar.urdf.xacro (robot description, xacro)
@@ -1,7 +1,15 @@
 <?xml version="1.0"?>
 <robot xmlns:xacro="http://ros.org/wiki/xacro">
-  <!-- Generic 2D LiDAR: one fixed joint plus a placeholder cylinder. The frame name
-       must match the frame_id published by the LiDAR driver. -->
-  <xacro:macro name="lidar" params="name:=laser parent_link:=base_link radius:=0.035 height:=0.04 *origin">
+  <!-- Slamtec RPLIDAR C1 (datasheet C1M1-R2, rev 1.0).
+       The frame sits on the scan plane, at the rotation center; its name must match the
+       frame_id of the driver. Body: 55.6 x 55.6 x 23.1 mm base + 18.2 mm optical head,
+       total 41.3 mm; scan plane 29.8 mm above the bottom of the base. -->
+  <xacro:macro name="lidar" params="name:=laser parent_link:=base_link *origin">
+    <xacro:property name="base_side"   value="0.0556"/>
+    <xacro:property name="base_height" value="0.0231"/>
+    <xacro:property name="head_height" value="0.0182"/>
+    <xacro:property name="head_radius" value="0.025"/>   <!-- approx., not in the datasheet -->
+    <xacro:property name="scan_plane"  value="0.0298"/>  <!-- from the bottom of the base -->
+    <xacro:property name="mass"        value="0.110"/>
     <joint name="${name}_joint" type="fixed">
       <xacro:insert_block name="origin"/>
@@ -11,7 +19,7 @@
     <link name="${name}">
       <visual>
-        <origin xyz="0 0 0" rpy="0 0 0"/>
+        <origin xyz="0 0 ${base_height/2 - scan_plane}"/>
         <geometry>
-          <cylinder radius="${radius}" length="${height}"/>
+          <box size="${base_side} ${base_side} ${base_height}"/>
         </geometry>
         <material name="${name}_black">
@@ -19,4 +27,24 @@
         </material>
       </visual>
+      <visual>
+        <origin xyz="0 0 ${base_height + head_height/2 - scan_plane}"/>
+        <geometry>
+          <cylinder radius="${head_radius}" length="${head_height}"/>
+        </geometry>
+        <material name="${name}_black"/>
+      </visual>
+      <collision>
+        <origin xyz="0 0 ${(base_height + head_height)/2 - scan_plane}"/>
+        <geometry>
+          <box size="${base_side} ${base_side} ${base_height + head_height}"/>
+        </geometry>
+      </collision>
+      <inertial>
+        <origin xyz="0 0 ${(base_height + head_height)/2 - scan_plane}"/>
+        <mass value="${mass}"/>
+        <inertia ixx="${mass/12*(base_side**2 + (base_height + head_height)**2)}" ixy="0" ixz="0"
+                 iyy="${mass/12*(base_side**2 + (base_height + head_height)**2)}" iyz="0"
+                 izz="${mass/6*base_side**2}"/>
+      </inertial>
     </link>
   </xacro:macro>
